File: displays/displays.kicad_sch (KiCad schematic)
At the start: 105 parts, among them U10 TZ-H1010-RGB/A-BU08UF-TA1305N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, U11 TZ-H1010-RGB/A-BU08UF-TA1305N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, U12 TZ-H1010-RGB/A-BU08UF-TA1305N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, U13 TZ-H1010-RGB/A-BU08UF-TA1305N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, U14 TZ-H1010-RGB/A-BU08UF-TA1305N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, U15 TZ-H1010-RGB/A-BU08UF-TA1305N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, U16 TZ-H1010-RGB/A-BU08UF-TA1305N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, U17 TZ-H1010-RGB/A-BU08UF-TA1305N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, U18 TZ-H1010-RGB/A-BU08UF-TA1305N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, U19 TZ-H1010-RGB/A-BU08UF-TA1305N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, U2 TZ-H1010-RGB/A-BU08UF-TA1305N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, U20 TZ-H1010-RGB/A-BU08UF-TA1305N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, U21 TZ-H1010-RGB/A-BU08UF-TA1305N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, U22 TZ-H1010-RGB/A-BU08UF-TA1305N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, U23 TZ-H1010-RGB/A-BU08UF-TA1305N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, U24 TZ-H1010-RGB/A-BU08UF-TA1305N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, U25 TZ-H1010-RGB/A-BU08UF-TA1305N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, U26 TZ-H1010-RGB/A-BU08UF-TA1305N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, U27 TZ-H1010-RGB/A-BU08UF-TA1305N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, U28 TZ-H1010-RGB/A-BU08UF-TA1305N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, U29 TZ-H1010-RGB/A-BU08UF-TA1305N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, U3 TZ-H1010-RGB/A-BU08UF-TA1305N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, U30 TZ-H1010-RGB/A-BU08UF-TA1305N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, U31 TZ-H1010-RGB/A-BU08UF-TA1305N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, U32 TZ-H1010-RGB/A-BU08UF-TA1305N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, U33 TZ-H1010-RGB/A-BU08UF-TA1305N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, U34 TZ-H1010-RGB/A-BU08UF-TA1305N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, U35 TZ-H1010-RGB/A-BU08UF-TA1305N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, U36 TZ-H1010-RGB/A-BU08UF-TA1305N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, U37 TZ-H1010-RGB/A-BU08UF-TA1305N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, U38 TZ-H1010-RGB/A-BU08UF-TA1305N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, U39 TZ-H1010-RGB/A-BU08UF-TA1305N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, U4 TZ-H1010-RGB/A-BU08UF-TA1305N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, U40 TZ-H1010-RGB/A-BU08UF-TA1305N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, U41 TZ-H1010-RGB/A-BU08UF-TA1305N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, U42 TZ-H1010-RGB/A-BU08UF-TA1305N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, U43 TZ-H1010-RGB/A-BU08UF-TA1305N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, U44 PJ-320A-4P DIP, U45 TPA6132A2RTER, U46 74LVC2G17GV_C53954310, U47 74LVC2G17GV_C53954310, U48 74LVC2G17GV_C53954310, U5 TZ-H1010-RGB/A-BU08UF-TA1305N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, U6 TZ-H1010-RGB/A-BU08UF-TA1305N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, U7 TZ-H1010-RGB/A-BU08UF-TA1305N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, U8 TZ-H1010-RGB/A-BU08UF-TA1305N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, U9 TZ-H1010-RGB/A-BU08UF-TA1305N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

Commit message: updated board
Parts:
- C1, C10, C11, C12, C13, C14, C15, C16, C17, C18, C19, C2, C20, C21, C22, C23, C24, C25, C26, C27, C28, C29, C3, C30, C31, C32, C33, C34, C35, C36, C37, C38, C39, C4, C40, C41, C42, C5, C6, C7, C8, C9: footprint lcsc_footprints:C307380_C0201 -> lcsc_footprints:C1525_C0402; symbol lcsc_imported:CL03A104KO3NNNC -> lcsc_imported:100nF_(104)_±10%_16V; LCSC C307380 -> C1525
- C43, C44, C45, C47: footprint lcsc_footprints:C29266_C0402 -> lcsc_footprints:C52923_C0402; symbol lcsc_imported:1uF_(105)_±10%_16V -> lcsc_imported:1uF_(105)_±10%_25V; LCSC C29266 -> C52923; Manufacturer SAMSUNG(三星) -> (none)
- R1: value 500 -> 200; footprint lcsc_footprints:C6460545_R0402 -> lcsc_footprints:C25087_R0402; symbol lcsc_imported:RT0402FRE07500RL -> lcsc_imported:200Ω_(2000)_±1%; LCSC C6460545 -> C25087; Manufacturer YAGEO(国巨) -> (none)
Connections:
- no-connect marks 9 -> 11
Other:
- moved on the sheet: C43, C44, C45, C47
